File: Untitled.sch (EAGLE design)
At the start: 12 parts, among them IC1 ILD4001, IC2 ILD4001, IC3 ILD4001, IC4 74AHC1G125DBV, IC5 74AHC1G125DBV, U1 ATMEGA328P

Commit message: almost done
Parts:
- added D1, D2, D3: LED-RGB-CA-THRUCLEAR, SparkFun-LED:LED-RGB-CA-THRUCLEAR
- added JP2: (no value), SparkFun-Connectors:M04JST-PTH-VERT
- added JP3: M02JST-PTH-VERT, SparkFun-Connectors:M02JST-PTH-VERT
- added JP4: (no value), SparkFun-Connectors:M06LONGPADS
- added JP5: (no value), SparkFun-Connectors:M03X22X3_SILK_MALE_PTH
- added U$2: LM3480IM4, SparkFun-PowerIC:LM3480IM4
Connections:
- new net 3V: U$1.VDD, U$2.OUT
- new net MISO: U1.PB4(MISO)
- new net MOSI: U1.PB3(MOSI/OC2)
- new net N$1: JP2.1, U$1.ELE3
- new net N$2: JP2.2, U$1.ELE2
- new net N$3: JP2.3, U$1.ELE1
- new net N$4: JP2.4, U$1.ELE0
- new net RX: U1.PD0(RXD)
- new net SCK: U1.PB5(SCK)
- new net SCL: IC5A.I, U1.PC5(ADC5/SCL)
- new net SCLO: IC5A.O, U$1.SCL
- new net SDA: IC4A.I, U1.PC4(ADC4/SDA)
- new net SDAO: IC4A.O, U$1.SDA
- new net TX: U1.PD1(TXD)
- net BOUT: now also D1.BLUE_CATHODE, D2.BLUE_CATHODE, D3.BLUE_CATHODE
- net GND: now also IC4A.OE, IC5A.OE, JP3.2, U$1.VSS, U$2.GND
- net GOUT: now also D1.GREEN_CATHODE, D2.GREEN_CATHODE, D3.GREEN_CATHODE
- net ROUT: now also D1.RED_CATHODE, D2.RED_CATHODE, D3.RED_CATHODE
- net VCC: now also D1.ANODE, D2.ANODE, D3.ANODE, JP3.1, U$2.IN
Other:
- moved on the sheet: IC4

Commit message: rev1
Parts:
- added C1: (no value), SparkFun-Capacitors:CAP0805
Connections:
- removed net N$13: R4.1, U1.PC6(/RESET)
- new net N$5: C1.2, R4.1, U1.PC6(/RESET)
- new net RESET: C1.1, JP4.6, JP5.5
- net GND: now also JP4.1, JP4.2, JP5.6
- net MISO: now also JP5.1
- net MOSI: now also JP5.4
- net RX: now also JP4.5, U1.PD1(TXD); no longer U1.PD0(RXD)
- net SCK: now also JP5.3
- net TX: now also JP4.4, U1.PD0(RXD); no longer U1.PD1(TXD)
- net VCC: now also JP4.3, JP5.2, R4.2
Changed lines of the file:
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@@
 <part name="D2" library="SparkFun-LED" deviceset="LED-RGB-CA-THRU" device="CLEAR"/>
 <part name="D3" library="SparkFun-LED" deviceset="LED-RGB-CA-THRU" device="CLEAR"/>
+<part name="C1" library="SparkFun-Capacitors" deviceset="CAP" device="0805"/>
 </parts>
 <sheets>
@@
 <instance part="D2" gate="G$1" x="-76.2" y="109.22" rot="R180"/>
 <instance part="D3" gate="G$1" x="-76.2" y="93.98" rot="R180"/>
+<instance part="C1" gate="G$1" x="-58.42" y="78.74" rot="R90"/>
 </instances>
 <busses>
@@
 <junction x="66.04" y="22.86"/>
 <junction x="76.2" y="20.32"/>
-</segment>
-</net>
-<net name="N$13" class="0">
-<segment>
-<pinref part="U1" gate="G$1" pin="PC6(/RESET)"/>
-<pinref part="R4" gate="G$1" pin="1"/>
-<wire x1="-48.26" y1="78.74" x2="-40.64" y2="78.74" width="0.1524" layer="91"/>
-<junction x="-40.64" y="78.74"/>
-<junction x="-48.26" y="78.74"/>
-<wire x1="-48.26" y1="78.74" x2="-50.8" y2="78.74" width="0.1524" layer="91"/>
 </segment>
 </net>
@@
 <junction x="-86.36" y="124.46"/>
 </segment>
+<segment>
+<pinref part="JP5" gate="G$1" pin="2"/>
+<wire x1="109.22" y1="27.94" x2="111.76" y2="27.94" width="0.1524" layer="91"/>
+<label x="109.22" y="27.94" size="1.778" layer="95"/>
+</segment>
+<segment>
+<pinref part="R4" gate="G$1" pin="2"/>
+<wire x1="-48.26" y1="88.9" x2="-48.26" y2="91.44" width="0.1524" layer="91"/>
+<label x="-48.26" y="91.44" size="1.778" layer="95"/>
+<junction x="-48.26" y="88.9"/>
+</segment>
+<segment>
+<pinref part="JP4" gate="G$1" pin="3"/>
+<wire x1="99.06" y1="99.06" x2="96.52" y2="99.06" width="0.1524" layer="91"/>
+<label x="93.98" y="99.06" size="1.778" layer="95"/>
+<junction x="99.06" y="99.06"/>
+</segment>
 </net>
 <net name="GND" class="0">
@@
 <junction x="20.32" y="86.36"/>
 </segment>
+<segment>
+<pinref part="JP5" gate="G$1" pin="6"/>
+<wire x1="109.22" y1="22.86" x2="111.76" y2="22.86" width="0.1524" layer="91"/>
+<label x="109.22" y="22.86" size="1.778" layer="95"/>
+</segment>
+<segment>
+<pinref part="JP4" gate="G$1" pin="1"/>
+<wire x1="99.06" y1="104.14" x2="96.52" y2="104.14" width="0.1524" layer="91"/>
+<label x="93.98" y="104.14" size="1.778" layer="95"/>
+<junction x="99.06" y="104.14"/>
+</segment>
+<segment>
+<pinref part="JP4" gate="G$1" pin="2"/>
+<wire x1="99.06" y1="101.6" x2="96.52" y2="101.6" width="0.1524" layer="91"/>
+<label x="93.98" y="101.6" size="1.778" layer="95"/>
+<junction x="99.06" y="101.6"/>
+</segment>
 </net>
 <net name="SDA" class="0">
@@
 <label x="10.16" y="25.4" size="1.778" layer="95"/>
 </segment>
+<segment>
+<pinref part="JP5" gate="G$1" pin="4"/>
+<wire x1="109.22" y1="25.4" x2="111.76" y2="25.4" width="0.1524" layer="91"/>
+<label x="109.22" y="25.4" size="1.778" layer="95"/>
+</segment>
 </net>
 <net name="MISO" class="0">
@@
 <label x="10.16" y="22.86" size="1.778" layer="95"/>
 </segment>
+<segment>
+<pinref part="JP5" gate="G$1" pin="1"/>
+<wire x1="93.98" y1="27.94" x2="91.44" y2="27.94" width="0.1524" layer="91"/>
+<label x="86.36" y="27.94" size="1.778" layer="95"/>
+</segment>
 </net>
 <net name="SCK" class="0">
@@
 <label x="10.16" y="20.32" size="1.778" layer="95"/>
 </segment>
+<segment>
+<pinref part="JP5" gate="G$1" pin="3"/>
+<wire x1="93.98" y1="25.4" x2="91.44" y2="25.4" width="0.1524" layer="91"/>
+<label x="86.36" y="25.4" size="1.778" layer="95"/>
+</segment>
 </net>
 <net name="RX" class="0">
+<segment>
+<pinref part="JP4" gate="G$1" pin="5"/>
+<wire x1="99.06" y1="93.98" x2="96.52" y2="93.98" width="0.1524" layer="91"/>
+<label x="93.98" y="93.98" size="1.778" layer="95"/>
+<junction x="99.06" y="93.98"/>
+</segment>
+<segment>
+<pinref part="U1" gate="G$1" pin="PD1(TXD)"/>
+<wire x1="7.62" y1="53.34" x2="10.16" y2="53.34" width="0.1524" layer="91"/>
+<label x="10.16" y="53.34" size="1.778" layer="95"/>
+</segment>
+</net>
+<net name="TX" class="0">
+<segment>
+<pinref part="JP4" gate="G$1" pin="4"/>
+<wire x1="99.06" y1="96.52" x2="96.52" y2="96.52" width="0.1524" layer="91"/>
+<label x="93.98" y="96.52" size="1.778" layer="95"/>
+<junction x="99.06" y="96.52"/>
+</segment>
 <segment>
 <pinref part="U1" gate="G$1" pin="PD0(RXD)"/>
@@
 </segment>
 </net>
-<net name="TX" class="0">
-<segment>
-<pinref part="U1" gate="G$1" pin="PD1(TXD)"/>
-<wire x1="7.62" y1="53.34" x2="10.16" y2="53.34" width="0.1524" layer="91"/>
-<label x="10.16" y="53.34" size="1.778" layer="95"/>
-</segment>
-</net>
+<net name="RESET" class="0">
+<segment>
+<pinref part="JP5" gate="G$1" pin="5"/>
+<wire x1="93.98" y1="22.86" x2="91.44" y2="22.86" width="0.1524" layer="91"/>
+<label x="86.36" y="22.86" size="1.778" layer="95"/>
+</segment>
+<segment>
+<pinref part="JP4" gate="G$1" pin="6"/>
+<wire x1="99.06" y1="91.44" x2="96.52" y2="91.44" width="0.1524" layer="91"/>
+<label x="91.44" y="91.44" size="1.778" layer="95"/>
+<junction x="99.06" y="91.44"/>
+</segment>
+<segment>
+<pinref part="C1" gate="G$1" pin="1"/>
+<wire x1="-63.5" y1="78.74" x2="-66.04" y2="78.74" width="0.1524" layer="91"/>
+<label x="-73.66" y="78.74" size="1.778" layer="95"/>
+<junction x="-63.5" y="78.74"/>
+</segment>
+</net>
+<net name="N$5" class="0">
+<segment>
+<pinref part="U1" gate="G$1" pin="PC6(/RESET)"/>
+<pinref part="R4" gate="G$1" pin="1"/>
+<wire x1="-40.64" y1="78.74" x2="-48.26" y2="78.74" width="0.1524" layer="91"/>
+<wire x1="-48.26" y1="78.74" x2="-55.88" y2="78.74" width="0.1524" layer="91"/>
+<pinref part="C1" gate="G$1" pin="2"/>
+<junction x="-55.88" y="78.74"/>
+<junction x="-48.26" y="78.74"/>
+<junction x="-40.64" y="78.74"/>
+</segment>
+</net>
