File: Untitled.brd (EAGLE design)
At the start: 100 x 80 mm, 12 parts, among them IC1 ILD4001, IC2 ILD4001, IC3 ILD4001, IC4 74AHC1G125DBV, IC5 74AHC1G125DBV, U1 ATMEGA328P

Commit message: almost done
Parts:
- added D1, D2, D3: LED-RGB-CA-THRUCLEAR, SparkFun-LED:LED-RGB-THRU
- added JP2: (no value), SparkFun-Connectors:JST-4-PTH-VERT
- added JP3: M02JST-PTH-VERT, SparkFun-Connectors:JST-2-PTH-VERT
- added JP4: (no value), SparkFun-Connectors:1X06_LONGPADS
- added JP5: (no value), SparkFun-Connectors:2X3
- added U$2: LM3480IM4, SparkFun-PowerIC:SOT23-3
- moved IC1 50.4 mm to (43.2, 56.6)
- moved IC3 50.4 mm to (43.2, 41.4)
- moved IC4 50.4 mm to (56.9, 58.4)
- moved IC5 50.4 mm to (51.1, 58.4)
- moved JP1 50.4 mm to (35.6, 56.4)
- moved R1 50.4 mm to (43.2, 59.2)
- moved R3 50.4 mm to (43.2, 43.9)
- moved R4 50.4 mm to (63.5, 49.3)
- moved U1 50.4 mm to (55.6, 48.8)
- moved IC2 50.4 mm to (43.2, 49.0)
- moved R2 50.4 mm to (43.2, 51.6)
- moved U$1 50.2 mm to (50.5, 64.8), turned to 90 degrees
Connections:
- new net 3V: U$1.20, U$2.1
- new net MISO: U1.16
- new net MOSI: U1.15
- new net N$1: JP2.1, U$1.11
- new net N$2: JP2.2, U$1.10
- new net N$3: JP2.3, U$1.9
- new net N$4: JP2.4, U$1.8
- new net RX: U1.30
- new net SCK: U1.17
- new net SCL: IC5.2, U1.28
- new net SCLO: IC5.4, U$1.2
- new net SDA: IC4.2, U1.27
- new net SDAO: IC4.4, U$1.3
- new net TX: U1.31
- net BOUT: now also D1.4, D2.4, D3.4
- net GND: now also IC4.1, IC5.1, JP3.2, U$1.6, U$2.3
- net GOUT: now also D1.3, D2.3, D3.3
- net ROUT: now also D1.1, D2.1, D3.1
- net VCC: now also D1.2, D2.2, D3.2, JP3.1, U$2.2
Routing:
- net ROUT: track 16.3 -> 35.3 mm
- net GOUT: track 15.5 -> 32.9 mm
- net BOUT: track 21.4 -> 35.9 mm
- net VCC: track 49.5 -> 63.2 mm
- net SDAO: track 0.00 -> 8.58 mm, vias 0 -> 2
- net SCLO: track 0.00 -> 7.38 mm, vias 0 -> 2
- net N$2: track 0.00 -> 7.34 mm
- net N$1: track 0.00 -> 6.66 mm
- net N$4: track 0.00 -> 6.59 mm
- net N$3: track 0.00 -> 6.45 mm
- net 3V: track 0.00 -> 4.92 mm
- net GND: track 0.00 -> 0.92 mm, vias 6 -> 7
Other:
- board size 100 x 80 mm -> 45.7 x 45.7 mm

Commit message: rev1
Parts:
- added C1: (no value), SparkFun-Capacitors:0805
Connections:
- removed net N$13: R4.1, U1.29
- new net N$5: C1.2, R4.1, U1.29
- new net RESET: C1.1, JP4.6, JP5.5
- net GND: now also JP4.1, JP4.2, JP5.6
- net MISO: now also JP5.1
- net MOSI: now also JP5.4
- net RX: now also JP4.5, U1.31; no longer U1.30
- net SCK: now also JP5.3
- net TX: now also JP4.4, U1.30; no longer U1.31
- net VCC: now also JP4.3, JP5.2, R4.2
Routing:
- net VCC: track 63.2 -> 141.9 mm
- net ROUT: track 35.3 -> 93.4 mm, vias 0 -> 1
- net GOUT: track 32.9 -> 83.8 mm, vias 0 -> 1
- net BOUT: track 35.9 -> 81.7 mm, vias 0 -> 2
- net RESET: track 0.00 -> 33.0 mm, vias 0 -> 2
- net SCL: track 0.00 -> 27.9 mm, vias 0 -> 2
- net MOSI: track 0.00 -> 25.4 mm
- net SDA: track 0.00 -> 14.3 mm
- net MISO: track 0.00 -> 13.6 mm
- net SCK: track 0.00 -> 13.3 mm
- net RX: track 0.00 -> 11.6 mm
- net TX: track 0.00 -> 10.6 mm
- net N$5: track 0.00 -> 7.92 mm
- net GND: track 0.92 -> 7.69 mm
- net N$13: track 2.73 -> 0.00 mm

Commit message: Fixed RGB LED spacing
RGB LEDs now have spaces between pads. Added 4 capacitive sense channel
breakouts.
Parts:
- added JP6: (no value), SparkFun-Connectors:JST-4-PTH-VERT
- D1, D2, D3: device SparkFun-LED:LED-RGB-THRU -> SparkFun-LED-fix:LED-RGB-THRU
- moved JP2 5.07 mm to (55.8, 69.5)
Connections:
- new net N$13: JP6.2, U$1.14
- new net N$14: JP6.3, U$1.13
- new net N$15: JP6.4, U$1.12
- new net N$6: JP6.1, U$1.15
Routing:
- net N$6: track 0.00 -> 9.58 mm
- net GND: track 7.69 -> 16.2 mm, vias 7 -> 11
- net N$13: track 0.00 -> 7.92 mm
- net N$14: track 0.00 -> 6.16 mm
- net N$15: track 0.00 -> 4.16 mm
- net N$1: track 6.66 -> 3.39 mm
- net N$2: track 7.34 -> 4.77 mm
- net N$4: track 6.59 -> 9.01 mm
Other:
- board text added: "<3 -Swiss"
